File: HBDV3.kicad_sch (KiCad schematic)
At the start: 0 parts

Commit message: big update, half done
Parts:
- added C1, C2: 2.2uF, Capacitor_SMD:C_0805_2012Metric_Pad1.18x1.45mm_HandSolder, symbol Device:C
- added C3, C5, C7: 0.1uF, Capacitor_SMD:C_0805_2012Metric_Pad1.18x1.45mm_HandSolder, symbol Device:C
- added C4: 10uF, Capacitor_SMD:C_0805_2012Metric_Pad1.18x1.45mm_HandSolder, symbol Device:C
- added C6: 100uF, Library:CP_Radial_D6.3mm_H_12.5mm_P2.50mm_Würth, symbol Device:C_Polarized_US
- added D1, D2, D5: QH05BZ600, Package_TO_SOT_SMD:TO-263-2, symbol New_Library:QH05BZ600
- added D3, D4: TSD18DYFRQ1, Diode_SMD:D_SOD-323_HandSoldering, symbol Device:D_Zener
- added J2: RJ45, symbol Connector:RJ45
- added J3: 6P4C, symbol Connector:6P4C
- added R10, R11, R4: 10k, Resistor_SMD:R_1206_3216Metric_Pad1.30x1.75mm_HandSolder, symbol Device:R
- added R2, R5, R6, R7, R8, R9: 10, Resistor_SMD:R_2512_6332Metric_Pad1.40x3.35mm_HandSolder, symbol Device:R
- added R3: 1, Resistor_SMD:R_2512_6332Metric_Pad1.40x3.35mm_HandSolder, symbol Device:R
- added U1: (no value), Library:DSO14-300mil-adapter, symbol New_Library:2EDR6258X-DSO-14-300-mil
Connections:
- new net: D1.1 (C), R5.2, R6.2
- new net: R4.2, U1.6 (STP/DTC)
- new net: D5.1 (C), R7.2, R8.2
- new net: D2.3 (A), R3.2
- new net +16.5V: C2.1, C3.1, C4.1, C5.1, C6.1, R3.1, U1.11 (VDDB), U1.3 (VDDI), U1.8 (VDDI)
- new net A_HIN: U1.1 (INA)
- new net A_LIN: U1.2 (INB)
- new net ENABLE: U1.5 (EN)
- new net GND: C3.2, C4.2, C6.2, R4.1, U1.4 (GNDI)
- new net GNDA: C1.2, C7.2, D3.2 (A), R11.2, U1.12 (GNDA)
- new net GNDB: C2.2, C5.2, D4.2 (A), R10.2, U1.9 (GNDB)
- new net OUTA: R2.1, R5.1, R6.1, U1.13 (OUTA)
- new net OUTB: R7.1, R8.1, R9.1, U1.10 (OUTB)
- new net VDDA: C1.1, C7.1, D2.1 (C), U1.14 (VDDA)
- new net VOUTA: D1.3 (A), D3.1 (K), R11.1, R2.2
- new net VOUTB: D4.1 (K), D5.3 (A), R10.1, R9.2
Other:
- note added: "Boot-strap and output supply bypass caps bypass caps min rec.: 20 x C_iss (30 nF) of mosfet (SemiQ GCMX005A120S7B1) => 600 nF -> approx 1 uF ceramics have less C under DC bias therefore -> 2.2 uF"
- note added: "Dead-time R_DTC 10 ns x 10 k => 100 ns"
- note added: "Gate resistors 5 ohm turn off 10 ohm turn on ultra fast turn off diode (trr = 10 ns)"
- note added: "Power bypass caps bulk and close proxim."
- note added: "TVS Zener min. 18.5V breakdown G-S pull down"

Commit message: Full schematic
Parts:
- removed J3: 6P4C, symbol Connector:6P4C
- added C10, C13, C14: 0.1uF, Capacitor_SMD:C_0805_2012Metric_Pad1.18x1.45mm_HandSolder, symbol Device:C
- added C11, C12: 2.2uF, Capacitor_SMD:C_0805_2012Metric_Pad1.18x1.45mm_HandSolder, symbol Device:C
- added C8: 100uF, Library:CP_Radial_D6.3mm_H_12.5mm_P2.50mm_Würth, symbol Device:C_Polarized_US
- added C9: 10uF, Capacitor_SMD:C_0805_2012Metric_Pad1.18x1.45mm_HandSolder, symbol Device:C
- added D10, D9: TSD18DYFRQ1, Diode_SMD:D_SOD-323_HandSoldering, symbol Device:D_Zener
- added D6, D7, D8: QH05BZ600, Package_TO_SOT_SMD:TO-263-2, symbol New_Library:QH05BZ600
- added J1: Screw_Terminal_01x02 PWR, symbol Connector:Screw_Terminal_01x02
- added J3: RJ45 IN, symbol Connector:RJ45
- added J4: RJ45 OUT, symbol Connector:RJ45
- added J5, J6: Screw_Terminal_01x04, symbol Connector:Screw_Terminal_01x04
- added R12, R20, R21: 10k, Resistor_SMD:R_1206_3216Metric_Pad1.30x1.75mm_HandSolder, symbol Device:R
- added R13, R14, R15, R16, R17, R18: 10, Resistor_SMD:R_2512_6332Metric_Pad1.40x3.35mm_HandSolder, symbol Device:R
- added R19: 1, Resistor_SMD:R_2512_6332Metric_Pad1.40x3.35mm_HandSolder, symbol Device:R
- added U2: (no value), Library:DSO14-300mil-adapter, symbol New_Library:2EDR6258X-DSO-14-300-mil
- J2: value RJ45 -> RJ45 PWR
Connections:
- net +16.5V: now also J2.2, J2.4, J2.6, J2.8, C10.1, C11.1, C13.1, C8.1, C9.1, J1.2 (Pin_2), R19.1, U2.11 (VDDB), U2.3 (VDDI), U2.8 (VDDI)
- net ENABLE: now also J3.5, J4.5, U2.5 (EN)
- net GND: now also J2.1, J2.3, J2.5, J2.7, C10.2, C8.2, C9.2, J1.1 (Pin_1), R12.1, U2.4 (GNDI)
- net GNDA: now also J5.2 (Pin_2)
- net GNDB: now also J5.4 (Pin_4)
- net VOUTA: now also J5.1 (Pin_1)
- net VOUTB: now also J5.3 (Pin_3)
- net A_HIN renamed Phase 0
- net Phase 0: now also J3.1, J4.3, U2.2 (INB)
- net A_LIN renamed Phase 180
- net Phase 180: now also J3.2, J4.4, U2.1 (INA)
- new net: D8.1 (C), R16.2, R17.2
- new net: R12.2, U2.6 (STP/DTC)
- new net: D7.1 (C), R13.2, R14.2
- new net: D6.3 (A), R19.2
- new net GNDA_B: C12.2, C14.2, D9.2 (A), J6.2 (Pin_2), R20.2, U2.12 (GNDA)
- new net GNDB_B: C11.2, C13.2, D10.2 (A), J6.4 (Pin_4), R21.2, U2.9 (GNDB)
- new net OUTA_B: R13.1, R14.1, R15.1, U2.13 (OUTA)
- new net OUTB_B: R16.1, R17.1, R18.1, U2.10 (OUTB)
- new net Phase 270: J3.4, J4.2
- new net Phase 90: J3.3, J4.1
- new net VDDA_B: C12.1, C14.1, D6.1 (C), U2.14 (VDDA)
- new net VOUTA_B: D7.3 (A), D9.1 (K), J6.1 (Pin_1), R15.2, R20.1
- new net VOUTB_B: D10.1 (K), D8.3 (A), J6.3 (Pin_3), R18.2, R21.1
- no-connect marks 0 -> 6
Other:
- note added: "Control Signal input and control signal output to connect to second board"
- note added: "Gate Driver A"
- note added: "Gate Driver B"
- note added: "Output to MOSFETs for driver A and B"
- note added: "Power RJ45 alternating +16.5V / GND to reduce inductance Backup screw terminal"
- moved on the sheet: C1, C2, C3, C4, C5, C6, C7, D1, D2, D3, D4, D5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
