File: HBDV3.kicad_sch (KiCad schematic)
At the start: 52 parts, among them J1 Screw_Terminal_01x02 PWR, J2 RJ45 PWR, J3 RJ45 IN, J4 RJ45 OUT, J5 Screw_Terminal_01x04, J6 Screw_Terminal_01x04

Commit message: Updated component values
Parts:
- removed R10: 10k, Resistor_SMD:R_1206_3216Metric_Pad1.30x1.75mm_HandSolder, symbol Device:R
- removed R13: 10, Resistor_SMD:R_2512_6332Metric_Pad1.40x3.35mm_HandSolder, symbol Device:R
- added R12, R24: 2k, Resistor_SMD:R_1206_3216Metric_Pad1.30x1.75mm_HandSolder, symbol Device:R
- added R20, R3, R4: 2, Resistor_SMD:R_2512_6332Metric_Pad1.40x3.35mm_HandSolder, symbol Device:R
- added R22: 1, Resistor_SMD:R_2512_6332Metric_Pad1.40x3.35mm_HandSolder, symbol Device:R
- J1: renamed from J2; footprint (none) -> Library:RJ45_E5J8800LJG2L; Digikey (none) -> https://www.digikey.ca/en/products/detail/pulse-electronics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
- J2: renamed from J1; footprint (none) -> Library:Phoenix_2p_push_terminal; Digikey (none) -> https://www.digikey.ca/en/products/detail/phoenix-contact/1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
- J3, J4: footprint (none) -> Library:RJ45_E5J8800LJG2L; Digikey (none) -> https://www.digikey.ca/en/products/detail/pulse-electronics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
- J5, J6: value Screw_Terminal_01x04 -> push_Terminal_01x04; footprint (none) -> Library:Phoenix_4p_push_terminal; Digikey (none) -> https://www.digikey.ca/en/products/detail/phoenix-contact/1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
- R10: renamed from R3; Digikey https://www.digikey.ca/en/products/detail/vishay-dale/CRCW2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 -> https://www.digikey.ca/en/products/detail/bourns-inc/CRS251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
- R11: value 10k -> 2k; Digikey https://www.digikey.ca/en/products/detail/vishay-dale/RCS120610K0FKEA/10059629 -> https://www.digikey.ca/en/products/detail/vishay-dale/RCS12062K00FKEA/10059676
- R14, R15, R16, R17, R18, R2, R5, R6, R7, R8, R9: value 10 -> 2; Digikey https://www.digikey.ca/en/products/detail/bourns-inc/CHP251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 -> https://www.digikey.ca/en/products/detail/vishay-dale/CRCW2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
- R19: value 1 -> 2; Digikey https://www.digikey.ca/en/products/detail/vishay-dale/CRCW25121R00FKEGHP/2222061 -> https://www.digikey.ca/en/products/detail/vishay-dale/CRCW25122R00FKEGHP/2229396
- R21: value 10k -> 2; footprint Resistor_SMD:R_1206_3216Metric_Pad1.30x1.75mm_HandSolder -> Resistor_SMD:R_2512_6332Metric_Pad1.40x3.35mm_HandSolder; Digikey https://www.digikey.ca/en/products/detail/vishay-dale/RCS12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 -> https://www.digikey.ca/en/products/detail/vishay-dale/CRCW2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
- R23: renamed from R20; value 10k -> 2k; Digikey https://www.digikey.ca/en/products/detail/vishay-dale/RCS120610K0FKEA/10059629 -> https://www.digikey.ca/en/products/detail/vishay-dale/RCS12062K00FKEA/10059676
- renumbered C6 to C1, C4 to C2, C2 to C4, C1 to C5, C5 to C6, D2 to D1, D1 to D2, D5 to D3, D3 to D4, D4 to D5, R4 to R1, R12 to R13
Connections:
- net +16.5V: now also R22.1; no longer R19.1
- net GNDA: now also J5.3 (Pin_3); no longer J5.2 (Pin_2)
- net GNDA_B: now also J6.3 (Pin_3); no longer J6.2 (Pin_2)
- net GNDB: now also J5.2 (Pin_2), R12.2; no longer J5.4 (Pin_4)
- net GNDB_B: now also J6.2 (Pin_2), R24.2; no longer J6.4 (Pin_4), R21.2
- net OUTA: now also R3.1, R4.1; no longer R6.1
- net OUTA_B: now also R16.1, R17.1
- net OUTB: now also R6.1
- net OUTB_B: now also R19.1, R21.1, R20.1; no longer R16.1, R17.1
- net VOUTA: now also J5.4 (Pin_4), R5.2, R4.2; no longer J5.1 (Pin_1), R2.2
- net VOUTA_B: now also J6.4 (Pin_4), R16.2, R17.2; no longer J6.1 (Pin_1), R15.2
- net VOUTB: now also J5.1 (Pin_1), R8.2, R12.1; no longer J5.3 (Pin_3)
- net VOUTB_B: now also J6.1 (Pin_1), R21.2, R20.2, R24.1; no longer J6.3 (Pin_3), R18.2, R21.1
- net at D7.1 (C), R14.2: now also R15.2
- net at R19.2: now also D8.1 (C), R18.2; no longer D6.3 (A)
- net at D3.1 (C), R7.2: now also R6.2; no longer R8.2
- new net: D6.3 (A), R22.2
- new net: D2.1 (C), R2.2, R3.2
Other:
- note added: "Gate resistors 1 ohm turn off 2 ohm turn on PARALLEL RES OPTIONAL ultra fast turn off diode (trr = 10 ns)"
- note removed: "Gate resistors 5 ohm turn off 10 ohm turn on ultra fast turn off diode (trr = 10 ns)"
